File: HW/KiCad/AETS/AETS.kicad_sch (KiCad schematic)
At the start: 27 parts, among them J1 USB_C_Receptacle_USB2.0, J2 BANANA SOCKETS, Q1 DMP3098LQ-7, Q2 BC857BW,115, Q3 SI2369BDS-T1-GE3

Commit message: first commit
Parts:
- removed C2: 100nF, Capacitor_SMD:C_0805_2012Metric, symbol Device:C
- removed D1: TPD2S017DBVR, EMC_ComConv:SOT95P280X145-6N, symbol EMC_ComConv:TPD2S017DBVR
- removed D2, D3: D_Schottky, symbol Device:D_Schottky
- removed D4: 30V, symbol Device:D_Zener
- removed J1: USB_C_Receptacle_USB2.0, EMC_ComConv:USB4500030A, symbol Connector:USB_C_Receptacle_USB2.0
- removed J2: BANANA SOCKETS, symbol Connector:Screw_Terminal_01x02
- removed Q1: DMP3098LQ-7, Package_TO_SOT_SMD:SOT-23, symbol Device:Q_PMOS_GSD
- removed Q2: BC857BW,115, EMC_ComConv:SOT65P210X110-3N, symbol EMC_ComConv:BC857BW,115
- removed Q3: SI2369BDS-T1-GE3, EMC_ComConv:SOT95P237X112-3N, symbol EMC_ComConv:SI2369BDS-T1-GE3
- removed R1: 100k, Resistor_SMD:R_0805_2012Metric, symbol Device:R
- removed R10, R11, R12: 10k, Resistor_SMD:R_0805_2012Metric, symbol Device:R
- removed R4: 1k5, Resistor_SMD:R_0805_2012Metric, symbol Device:R
- removed R5, R6: 10R, Resistor_SMD:R_0805_2012Metric, symbol Device:R
- added C11, C22, C23, C27, C28, C30, C31, C6: 100nF, Capacitor_SMD:C_0805_2012Metric, symbol Device:C
- added C12, C13: 47p, Capacitor_SMD:C_0805_2012Metric, symbol Device:C
- added C14, C15, C18, C19, C21, C7: 100nF, Capacitor_SMD:C_0603_1608Metric, symbol Device:C_Small
- added C16: 10nF, Capacitor_SMD:C_0805_2012Metric, symbol Device:C
- added C20, C24, C25, C26: 4,7uF, Capacitor_SMD:C_1210_3225Metric, symbol Device:C
- added C29, C32: 68uF, AETS:EEEHP1H4R7P, symbol AETS:EEE-FP1C680AL
- added C8: 4,7nF, Capacitor_SMD:C_0805_2012Metric, symbol Device:C
- added D17: VS-10BQ015HM3_5BT, AETS:DIOM5436X244N, symbol AETS:VS-10BQ015HM3_5BT
- added D3: 1.5B18CA-M3/H, AETS:DIOM5436X244N, symbol EMC_ComConv:GG060305100N2P
- added F1: ERB-RD0R50X, Resistor_SMD:R_0402_1005Metric, symbol Device:Fuse_Small
- added IC1: MCP2542WFD-E_SN, AETS:SOIC127P600X175-8N, symbol EMC_ComConv:MCP2542WFD-E_SN
- added IC2: M24512-DRMN8TP_K, AETS:SOIC127P600X175-8N, symbol AETS:M24512-DRMN8TP_K
- added IC3: STM32G474RET6, AETS:QFP50P1200X1200X160-64N, symbol EMC_ComConv:STM32G474RET6
- added IC4: LD29080DT50R, AETS:L4931CDT50TR, symbol AETS:L4931CDT50-TR
- added IC5, IC6: TPS7B6933DBVR, AETS:SOT95P280X145-5N, symbol EMC_ComConv:TPS7B6950QDBVRQ1
- added J1: Conn_01x14_Pin, Connector_PinHeader_2.54mm:PinHeader_1x14_P2.54mm_Vertical, symbol Connector:Conn_01x14_Pin
- added J6: DC-10A FC68148, AETS:DC10AFC68148, symbol Connector:Barrel_Jack_Switch
- added R14: 100k, Resistor_SMD:R_0805_2012Metric, symbol Device:R
- added R15: 10k, Resistor_SMD:R_0805_2012Metric, symbol Device:R
- added R16: 10R, Resistor_SMD:R_0805_2012Metric, symbol Device:R
- added R17: 10k, Resistor_SMD:R_0603_1608Metric, symbol Device:R
- added R18, R19: 2k2, Resistor_SMD:R_0805_2012Metric, symbol Device:R
- added RV5, RV6: AVR-M1608C270KTACB, AETS:VARC1608X90N, symbol AETS:AVR-M1608C270KTACB
- added Y1: Crystal_GND24, AETS:ECS4001833JGNTR3, symbol Device:Crystal_GND24
- C1: value 100n -> 100nF; footprint (none) -> Capacitor_SMD:C_0805_2012Metric
- C3: value 10nF -> 100nF
- C4: value 10nF -> 10pF
- C5: value 100nF -> 10pF; footprint Capacitor_SMD:C_0805_2012Metric -> Capacitor_SMD:C_0603_1608Metric
- FB1: footprint (none) -> Resistor_SMD:R_0805_2012Metric_Pad1.20x1.40mm_HandSolder
- R2: value 5k1 -> 0R; footprint Resistor_SMD:R_0805_2012Metric -> Resistor_SMD:R_0603_1608Metric
- R3: value 5k1 -> 1M; footprint Resistor_SMD:R_0805_2012Metric -> Resistor_SMD:R_0603_1608Metric; now not fitted
- R7: value 10k -> 60,4R
- R8: value 100k -> 60,4R
- R9: value 11k -> 10k; footprint Resistor_SMD:R_0805_2012Metric -> Resistor_SMD:R_0603_1608Metric
Connections:
- net +3.3V: now also R9.2, C14.1, C15.2, C19.2, C21.1, C29.1 (+), C30.1, C6.1, IC1.5 (VIO), IC3.1 (VBAT), IC3.16 (VDD_1), IC3.32 (VDD_2), IC3.48 (VDD_3), IC3.64 (VDD_4), IC5.5 (OUT), J1.1 (Pin_1), R16.2, R18.2, R19.2
- net DIAG_VBUS: now also C16.1, IC3.12 (PA0), R14.2, R15.1; no longer C4.1, R8.2, R9.1
- net GND: now also C5.2, C11.2, C12.2, C13.1, C14.2, C15.1, C16.2, C18.1, C19.1, C20.2, C21.2, C22.2, C23.2, C24.2, C25.2, C26.2, C27.2, C28.2, C29.2 (-), C30.2, C31.2, C32.2 (-), C6.2, C7.1, C8.2, D3.1 (K1), IC1.2 (VSS), IC2.1 (E0), IC2.2 (E1), IC2.3 (E2), IC2.4 (VSS), IC2.7 (~{WC}), IC3.15 (VSS_1), IC3.27 (VSSA), IC3.31 (VSS_2), IC3.47 (VSS_3), IC3.63 (VSS_4), IC4.2 (GND), IC5.3 (GND_1), IC5.4 (GND_2), IC6.3 (GND_1), IC6.4 (GND_2), J1.13 (Pin_13), J1.2 (Pin_2), J6.2, J6.3, R15.2, R17.1, RV5.1, RV6.2, Y1.2, Y1.4; no longer R2.1, R3.1, R7.1, R9.2
- net USB_DIS: now also IC3.44 (PA10); no longer R7.2
- net USB_DM: now also IC3.45 (PA11)
- net USB_DP: now also IC3.46 (PA12)
- net at FB1.1: now also D17.1 (K), D3.2 (K2)
- net CC1: no longer names the net of R2.2
- net CC1: now also C4.1, Y1.1
- net CC2 renamed OSC_IN
- net OSC_IN: now also C5.1, IC3.5 (PF0-OSC_IN), Y1.3
- net VBUS-USB-C: no longer names the net of C3.1
- net VBUS-USB-C: now also D17.2 (A), F1.2
- new net: C11.1, IC2.8 (VCC), R16.1
- new net: C8.1, R7.2, R8.1
- new net: IC3.61 (PB8-BOOT0), R17.2
- new net: F1.1, J6.1
- new net +12V: C20.1, C22.1, FB1.2, IC4.1 (INPUT), R14.1
- new net +3.3VA: C18.2, C31.1, C32.1 (+), IC3.29 (VDDA), IC6.5 (OUT)
- new net +5V: C1.1, C23.1, C24.1, C25.1, C26.1, C27.1, C28.1, IC1.3 (VDD), IC4.3 (OUTPUT), IC5.1 (IN), IC6.1 (IN), J1.14 (Pin_14)
- new net ADC_RELAY1_CURRENT: IC3.8 (PC0)
- new net ADC_RELAY2_CURRENT: IC3.9 (PC1)
- new net ADC_RELAY3_CURRENT: IC3.10 (PC2)
- new net ADC_RELAY4_CURRENT: IC3.11 (PC3)
- new net CANH: C12.1, IC1.7 (CANH), R7.1, RV5.2
- new net CANL: C13.2, IC1.6 (CANL), R8.2, RV6.1
- new net CAN_RXD: IC1.4 (RXD), IC3.34 (PB12)
- new net CAN_STB: IC1.8 (STBY), IC3.33 (PB11)
- new net CAN_TXD: IC1.1 (TXD), IC3.35 (PB13)
- new net EEPROM_SCL: IC2.5 (SDA), IC3.40 (PC8), R19.1
- new net EEPROM_SDA: IC2.6 (SCL), IC3.41 (PC9), R18.1
- new net Encoder_A: IC3.42 (PA8)
- new net Encoder_B: IC3.43 (PA9)
- new net Encoder_SW: IC3.30 (PB10)
- new net MCU_BUZZER: IC3.17 (PA3)
- new net MCU_GPIO_MOSFET1: IC3.38 (PC6)
- new net MCU_GPIO_MOSFET2: IC3.36 (PB14)
- new net MCU_GPIO_MUX1: IC3.39 (PC7)
- new net MCU_GPIO_MUX2: IC3.37 (PB15)
- new net MCU_GPIO_RELAY1: IC3.26 (PB2)
- new net MCU_GPIO_RELAY2: IC3.25 (PB1)
- new net MCU_GPIO_RELAY3: IC3.24 (PB0)
- new net MCU_GPIO_RELAY4: IC3.23 (PC5)
- new net MCU_TRIGGER_OUT: IC3.18 (PA4)
- new net NRST: C7.2, IC3.7 (PG10-NRST), R9.1
- new net OLED_CS: IC3.20 (PA6)
- new net OLED_MOSI: IC3.21 (PA7)
- new net OLED_SCL: IC3.19 (PA5)
- new net OSC_OUT: IC3.6 (PF1-OSC_OUT), R2.1, R3.1
- new net PA15: IC3.51 (PA15), J1.3 (Pin_3)
- new net PB3: IC3.56 (PB3), J1.8 (Pin_8)
- new net PB4: IC3.57 (PB4), J1.9 (Pin_9)
- new net PB5: IC3.58 (PB5), J1.10 (Pin_10)
- new net PB6: IC3.59 (PB6), J1.11 (Pin_11)
- new net PB7: IC3.60 (PB7), J1.12 (Pin_12)
- new net PC10: IC3.52 (PC10), J1.4 (Pin_4)
- new net PC11: IC3.53 (PC11), J1.5 (Pin_5)
- new net PC12: IC3.54 (PC12), J1.6 (Pin_6)
- new net PD2: IC3.55 (PD2), J1.7 (Pin_7)
- new net SWCLK: IC3.50 (PA14)
- new net SWDIO: IC3.49 (PA13)
- no-connect marks 2 -> 8
Other:
- added sheet Connections (Connections.kicad_sch)
- added sheet MOSFET_PART (MOSFET.kicad_sch)
- added sheet RELAY_PART (RELAYS.kicad_sch)
- added sheet UI (UI.kicad_sch)
- note added: "100pF Cbus"
- note added: "CAN"
- note added: "CONNECTION PART"
- note added: "Crystal"
- note added: "EEPROM"
- note added: "MCU"
- note added: "MOSFET PART"
- note added: "RELAY PART"
- note added: "UI PART"
- note added: "tr=0,8473*2200*100*10^-12 = 187 nS"
- note removed: "USB-C Connector with protection"
- note removed: "bacha na footprint!!!!"
- moved on the sheet: FB1
