File: HW/KiCad/AETS/UI.kicad_sch (KiCad schematic)
At the start: 13 parts, among them J5 B6B-XH-A, J6 B5B-XH-A__LF__SN_, Q15 NPN

Commit message: aa
Parts:
- DS1: now fitted
Changed lines of the file:
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@@
 	(wire
 		(pts
-			(xy 38.1 74.93) (xy 44.45 74.93)
+			(xy 39.37 74.93) (xy 44.45 74.93)
 		)
 		(stroke
@@
 	(symbol
 		(lib_id "power:GND")
-		(at 38.1 74.93 270)
+		(at 39.37 74.93 270)
 		(unit 1)
 		(exclude_from_sim no)
@@
 		(fields_autoplaced yes)
 		(property "Reference" "#PWR0107"
-			(at 31.75 74.93 0)
+			(at 33.02 74.93 0)
 			(effects
 				(font
@@
 		)
 		(property "Value" "GND"
-			(at 34.29 74.9299 90)
+			(at 35.56 74.9299 90)
 			(effects
 				(font
@@
 		)
 		(property "Footprint" ""
-			(at 38.1 74.93 0)
+			(at 39.37 74.93 0)
 			(effects
 				(font
@@
 		)
 		(property "Datasheet" ""
-			(at 38.1 74.93 0)
+			(at 39.37 74.93 0)
 			(effects
 				(font
@@
 		)
 		(property "Description" ""
-			(at 38.1 74.93 0)
+			(at 39.37 74.93 0)
 			(effects
 				(font
@@
 		(exclude_from_sim no)
 		(in_bom yes)
-		(on_board no)
-		(dnp yes)
+		(on_board yes)
+		(dnp no)
 		(fields_autoplaced yes)
 		(property "Reference" "DS1"
